Commit message: Added target model.  Rebuilt Kentland Farm world using Gazebo.

File: src/mbzirc_gazebo/worlds/kentland_farm.world.xacro (robot description, xacro)
@@ -1,36 +1,54 @@
-<?xml version="1.0" ?>
-<sdf version="1.4">
-  <world name="default" xmlns:xacro="http://ros.org/wiki/xacro">
-    <!-- A global light source -->
-    <include>
-      <uri>model://sun</uri>
-    </include>
-    <!-- A ground plane -->
-    <include>
-      <uri>model://ground_plane</uri>
-    </include>
-    <gui>
-      <camera name="user_camera">
-        <pose>72 -32 4 0 0.3 ${3 * pi / 4}</pose>
-      </camera>
-    </gui>
-    <!-- Field -->
-    <model name="ground">
-      <pose>0 0 0 0 0 0</pose>
-      <static>true</static>
-      <link name="link">
-        <collision name="ground_collision">
+<?xml version='1.0'?>
+<sdf xmlns:xacro='http://www.ros.org/wiki/xacro' version='1.6'>
+  <world name='default'>
+    <xacro:property name='x' value='107.0' />
+    <xacro:property name='y' value='53.5' />
+    <light name='sun' type='directional'>
+      <cast_shadows>1</cast_shadows>
+      <pose frame=''>0 0 10 0 -0 0</pose>
+      <diffuse>0.8 0.8 0.8 1</diffuse>
+      <specular>0.1 0.1 0.1 1</specular>
+      <attenuation>
+        <range>1000</range>
+        <constant>0.9</constant>
+        <linear>0.01</linear>
+        <quadratic>0.001</quadratic>
+      </attenuation>
+      <direction>-0.5 0.5 -1</direction>
+    </light>
+    <model name='ground_plane'>
+      <static>1</static>
+      <link name='link'>
+        <collision name='collision'>
           <geometry>
-            <box>
-              <size>107.0 53.5 0.15</size>
-            </box>
+            <plane>
+              <normal>0 0 1</normal>
+              <size>${x} ${y}</size>
+            </plane>
           </geometry>
+          <surface>
+            <friction>
+              <ode>
+                <mu>100</mu>
+                <mu2>50</mu2>
+              </ode>
+              <torsional>
+                <ode/>
+              </torsional>
+            </friction>
+            <contact>
+              <ode/>
+            </contact>
+            <bounce/>
+          </surface>
+          <max_contacts>10</max_contacts>
         </collision>
-        <visual name="ground_visual">
+        <visual name='visual'>
+          <cast_shadows>0</cast_shadows>
           <geometry>
-            <box>
-              <size>107.0 53.5 0.15</size>
-              <!-- <size>160.0 80.0 0.15</size> -->
-            </box>
+            <plane>
+              <normal>0 0 1</normal>
+              <size>${x} ${y}</size>
+            </plane>
           </geometry>
           <material>
@@ -42,6 +60,74 @@
           </material>
         </visual>
+        <self_collide>0</self_collide>
+        <kinematic>0</kinematic>
+        <gravity>1</gravity>
       </link>
     </model>
+    <!-- Testing the automatic population of objects
+    <xacro:if value="1">
+      <population name="can_population1">
+        <model name="can1">
+          <include>
+            <static>true</static>
+            <uri>$(find mbzirc_gazebo)/models/target</uri>
+          </include>
+        </model>
+        <pose>0 0 0 0 0 0</pose>
+        <box>
+          <size>${x} ${y}</size>
+        </box>
+        <model_count>10</model_count>
+        <distribution>
+          <type>random</type>
+        </distribution>
+      </population>
+    </xacro:if> -->
+    <gravity>0 0 -9.8</gravity>
+    <magnetic_field>6e-06 2.3e-05 -4.2e-05</magnetic_field>
+    <atmosphere type='adiabatic'/>
+    <physics name='default_physics' default='0' type='ode'>
+      <max_step_size>0.001</max_step_size>
+      <real_time_factor>1</real_time_factor>
+      <real_time_update_rate>1000</real_time_update_rate>
+    </physics>
+    <scene>
+      <ambient>0.4 0.4 0.4 1</ambient>
+      <background>0.7 0.7 0.7 1</background>
+      <shadows>1</shadows>
+    </scene>
+    <spherical_coordinates>
+      <surface_model>EARTH_WGS84</surface_model>
+      <latitude_deg>0</latitude_deg>
+      <longitude_deg>0</longitude_deg>
+      <elevation>0</elevation>
+      <heading_deg>0</heading_deg>
+    </spherical_coordinates>
+    <state world_name='default'>
+      <sim_time>32 156000000</sim_time>
+      <real_time>32 268040396</real_time>
+      <wall_time>1466110903 721775684</wall_time>
+      <iterations>32156</iterations>
+      <model name='ground_plane'>
+        <pose frame=''>0 0 0 0 -0 0</pose>
+        <scale>1 1 1</scale>
+        <link name='link'>
+          <pose frame=''>0 0 0 0 -0 0</pose>
+          <velocity>0 0 0 0 -0 0</velocity>
+          <acceleration>0 0 0 0 -0 0</acceleration>
+          <wrench>0 0 0 0 -0 0</wrench>
+        </link>
+      </model>
+      <light name='sun'>
+        <pose frame=''>0 0 10 0 -0 0</pose>
+      </light>
+    </state>
+    <gui fullscreen='0'>
+      <camera name='user_camera'>
+        <pose frame=''>5 -5 2 0 0.275643 2.35619</pose>
+        <view_controller>orbit</view_controller>
+        <projection_type>perspective</projection_type>
+      </camera>
+    </gui>
   </world>
 </sdf>

Commit message: Added start area and drop area to Kentland Farm world.

File: src/mbzirc_gazebo/worlds/kentland_farm.world.xacro (robot description, xacro)
@@ -65,23 +65,12 @@
       </link>
     </model>
-    <!-- Testing the automatic population of objects
-    <xacro:if value="1">
-      <population name="can_population1">
-        <model name="can1">
-          <include>
-            <static>true</static>
-            <uri>$(find mbzirc_gazebo)/models/target</uri>
-          </include>
-        </model>
-        <pose>0 0 0 0 0 0</pose>
-        <box>
-          <size>${x} ${y}</size>
-        </box>
-        <model_count>10</model_count>
-        <distribution>
-          <type>random</type>
-        </distribution>
-      </population>
-    </xacro:if> -->
+    <model name='start_area'>
+      <xacro:include filename='$(find mbzirc_gazebo)/models/designation_area/model.sdf' />
+      <pose frame=''>${(x / 2) - 7} ${(-y / 2) + 7} 0 0 0 0</pose>
+    </model>
+    <model name='drop_area'>
+      <xacro:include filename='$(find mbzirc_gazebo)/models/designation_area/model.sdf' />
+      <pose frame=''>${(-x / 2) + 7} ${(y / 2) - 7} 0 0 0 0</pose>
+    </model>
     <gravity>0 0 -9.8</gravity>
     <magnetic_field>6e-06 2.3e-05 -4.2e-05</magnetic_field>
